File: esp32-canbus.sch (EAGLE design)
At the start: 59 parts, among them J1 PRPC006DBAN-M71RC, J2 USB-MICROB-3, U1 ESP32, U10 TPS62172DSGR, U3 MCP2515T-I/ML, U4 MCP2515T-I/ML, U5 MCP2515T-I/ML, U6 MCP2558FDT-H/MNY, U7 MCP2558FDT-H/MNY, U8 MCP2558FDT-H/MNY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

Commit message: Update board
Rout mode of the board and a few edits in the schematic
Connections:
- net !INT0: now also U1.GPIO16*/HS1_DATA4/U2RXD/EMAC_CLK_OUT; no longer U1.GPIO00*/ADC2_CH1/TOUCH1/RTC_GPIO11/CLK_OUT1/EMAC_TX_CLK
- net !INT2: now also U1.GPIO00*/ADC2_CH1/TOUCH1/RTC_GPIO11/CLK_OUT1/EMAC_TX_CLK; no longer U1.GPIO16*/HS1_DATA4/U2RXD/EMAC_CLK_OUT
- net A0: now also J1.12; no longer J1.9
- net A1: now also J1.11; no longer J1.10
- net A2: now also J1.10; no longer J1.11
- net A3: now also J1.9; no longer J1.12
Changed lines of the file:
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@@
 </segment>
 <segment>
-<pinref part="U1" gate="G$1" pin="GPIO16*/HS1_DATA4/U2RXD/EMAC_CLK_OUT"/>
-<wire x1="-63.5" y1="1.27" x2="-66.04" y2="1.27" width="0.1524" layer="91"/>
-<label x="-66.04" y="1.27" size="1.27" layer="95" rot="R180" xref="yes"/>
+<pinref part="U1" gate="G$1" pin="GPIO00*/ADC2_CH1/TOUCH1/RTC_GPIO11/CLK_OUT1/EMAC_TX_CLK"/>
+<wire x1="-63.5" y1="41.91" x2="-66.04" y2="41.91" width="0.1524" layer="91"/>
+<label x="-66.04" y="41.91" size="1.27" layer="95" rot="R180" xref="yes"/>
 </segment>
 </net>
@@
 </segment>
 <segment>
-<pinref part="U1" gate="G$1" pin="GPIO00*/ADC2_CH1/TOUCH1/RTC_GPIO11/CLK_OUT1/EMAC_TX_CLK"/>
-<wire x1="-63.5" y1="41.91" x2="-66.04" y2="41.91" width="0.1524" layer="91"/>
-<label x="-66.04" y="41.91" size="1.27" layer="95" rot="R180" xref="yes"/>
+<pinref part="U1" gate="G$1" pin="GPIO16*/HS1_DATA4/U2RXD/EMAC_CLK_OUT"/>
+<wire x1="-63.5" y1="1.27" x2="-66.04" y2="1.27" width="0.1524" layer="91"/>
+<label x="-66.04" y="1.27" size="1.27" layer="95" rot="R180" xref="yes"/>
 </segment>
 </net>
 <net name="A0" class="0">
+<segment>
+<pinref part="U1" gate="G$1" pin="GPIO32/32K_XP*/ADC1_CH4/TOUCH9/RTC_GPIO9"/>
+<wire x1="-63.5" y1="-24.13" x2="-66.04" y2="-24.13" width="0.1524" layer="91"/>
+<label x="-66.04" y="-24.13" size="1.27" layer="95" rot="R180" xref="yes"/>
+</segment>
+<segment>
+<pinref part="J1" gate="G$1" pin="12"/>
+<wire x1="-39.37" y1="52.07" x2="-41.91" y2="52.07" width="0.1524" layer="91"/>
+<label x="-39.37" y="52.07" size="1.27" layer="95" xref="yes"/>
+</segment>
+</net>
+<net name="A2" class="0">
+<segment>
+<pinref part="U1" gate="G$1" pin="GPIO25*/DAC_1/ADC2_CH8/RTC_GPIO6/EMAC_RXD0"/>
+<wire x1="-63.5" y1="-16.51" x2="-66.04" y2="-16.51" width="0.1524" layer="91"/>
+<label x="-66.04" y="-16.51" size="1.27" layer="95" rot="R180" xref="yes"/>
+</segment>
+<segment>
+<pinref part="J1" gate="G$1" pin="10"/>
+<wire x1="-41.91" y1="54.61" x2="-39.37" y2="54.61" width="0.1524" layer="91"/>
+<label x="-39.37" y="54.61" size="1.27" layer="95" xref="yes"/>
+</segment>
+</net>
+<net name="A1" class="0">
+<segment>
+<pinref part="U1" gate="G$1" pin="GPIO33/32K_XN*/ADC1_CH5/TOUCH8/RTC_GPIO8"/>
+<wire x1="-63.5" y1="-26.67" x2="-66.04" y2="-26.67" width="0.1524" layer="91"/>
+<label x="-66.04" y="-26.67" size="1.27" layer="95" rot="R180" xref="yes"/>
+</segment>
+<segment>
+<pinref part="J1" gate="G$1" pin="11"/>
+<wire x1="-57.15" y1="52.07" x2="-59.69" y2="52.07" width="0.1524" layer="91"/>
+<label x="-59.69" y="52.07" size="1.27" layer="95" rot="R180" xref="yes"/>
+</segment>
+</net>
+<net name="A3" class="0">
+<segment>
+<pinref part="U1" gate="G$1" pin="GPIO26*/DAC_2/ADC2_CH9/RTC_GPIO7/RMAC_RXD1"/>
+<wire x1="-63.5" y1="-19.05" x2="-66.04" y2="-19.05" width="0.1524" layer="91"/>
+<label x="-66.04" y="-19.05" size="1.27" layer="95" rot="R180" xref="yes"/>
+</segment>
 <segment>
 <pinref part="J1" gate="G$1" pin="9"/>
@@
 <label x="-59.69" y="54.61" size="1.27" layer="95" rot="R180" xref="yes"/>
 </segment>
-<segment>
-<pinref part="U1" gate="G$1" pin="GPIO32/32K_XP*/ADC1_CH4/TOUCH9/RTC_GPIO9"/>
-<wire x1="-63.5" y1="-24.13" x2="-66.04" y2="-24.13" width="0.1524" layer="91"/>
-<label x="-66.04" y="-24.13" size="1.27" layer="95" rot="R180" xref="yes"/>
-</segment>
 </net>
-<net name="A2" class="0">
-<segment>
-<pinref part="J1" gate="G$1" pin="11"/>
-<wire x1="-57.15" y1="52.07" x2="-59.69" y2="52.07" width="0.1524" layer="91"/>
-<label x="-59.69" y="52.07" size="1.27" layer="95" rot="R180" xref="yes"/>
-</segment>
-<segment>
-<pinref part="U1" gate="G$1" pin="GPIO25*/DAC_1/ADC2_CH8/RTC_GPIO6/EMAC_RXD0"/>
-<wire x1="-63.5" y1="-16.51" x2="-66.04" y2="-16.51" width="0.1524" layer="91"/>
-<label x="-66.04" y="-16.51" size="1.27" layer="95" rot="R180" xref="yes"/>
-</segment>
-</net>
-<net name="A1" class="0">
-<segment>
-<pinref part="J1" gate="G$1" pin="10"/>
-<wire x1="-41.91" y1="54.61" x2="-39.37" y2="54.61" width="0.1524" layer="91"/>
-<label x="-39.37" y="54.61" size="1.27" layer="95" xref="yes"/>
-</segment>
-<segment>
-<pinref part="U1" gate="G$1" pin="GPIO33/32K_XN*/ADC1_CH5/TOUCH8/RTC_GPIO8"/>
-<wire x1="-63.5" y1="-26.67" x2="-66.04" y2="-26.67" width="0.1524" layer="91"/>
-<label x="-66.04" y="-26.67" size="1.27" layer="95" rot="R180" xref="yes"/>
-</segment>
-</net>
-<net name="A3" class="0">
-<segment>
-<pinref part="J1" gate="G$1" pin="12"/>
-<wire x1="-39.37" y1="52.07" x2="-41.91" y2="52.07" width="0.1524" layer="91"/>
-<label x="-39.37" y="52.07" size="1.27" layer="95" xref="yes"/>
-</segment>
-<segment>
-<pinref part="U1" gate="G$1" pin="GPIO26*/DAC_2/ADC2_CH9/RTC_GPIO7/RMAC_RXD1"/>
-<wire x1="-63.5" y1="-19.05" x2="-66.04" y2="-19.05" width="0.1524" layer="91"/>
-<label x="-66.04" y="-19.05" size="1.27" layer="95" rot="R180" xref="yes"/>
-</segment>
-</net>

Commit message: Update board
Finish board layou, tweak a few things in schematic, and add documents
(ger ber files, pdf schematic)
Parts:
- added C30, C31: 0.1uF, Passives:CAP-0603
- added D1: NSR0530HT1G, ON Semiconductor:NSR0530HT1G
- added D2: LH R974-LP-1, Passives:LED-0805
- added JUMPER1, JUMPER2, JUMPER3: JUMPER-NO, Passives:JUMPER-NO
- added R10, R11, R12: 10k, Passives:RESISTOR-0603
- added R13: 1k, Passives:RESISTOR-0603
- added R14, R15, R16: 120, Passives:RESISTOR-0603
- added S1: TACTILE-SMD2, Passives:TACTILE-SMD2
- added U11: CP2104-F03-GM, Silicon Labs:CP2104-F03-GM
- C14, C2: value 18pF -> 10pF
- C15, C3: value 18pFF -> 10pF
- F1, F2: value (none) -> 0ZCJ0050AF2E; device Passives:PTC-1812 -> Passives:PTC-1206
- J2: value USB-MICROB-3 -> 10118192-0001LF
- L1: device Passives:INDUCTOR-0603 -> Passives:INDUCTOR-0402
- SH1: value RF-SHIELD -> BMI-S-102
- U2: value (none) -> SST26WF080BT-104I/NP
- renumbered U$1 to SH1
Connections:
- new net D_N: J2.D-, U11.D-
- new net D_P: J2.D+, U11.D+
- new net N$27: R10.1, U11.!RST
- new net N$28: D1.C, F2.1
- new net N$29: D2.C, R13.2
- new net N$31: JUMPER1.P$2, R14.1
- new net N$32: C31.1, U11.VPP
- new net N$34: JUMPER2.P$2, R15.1
- new net N$35: JUMPER3.P$2, R16.1
- new net PROGRAM: S1.3, U1.GPIO00*/ADC2_CH1/TOUCH1/RTC_GPIO11/CLK_OUT1/EMAC_TX_CLK
- new net VBUS: D1.A, J2.VBUS, R11.2
- net !INT2: now also U1.GPIO38/SENSOR_CAPN*/ADC_PRE_AMP/ADC1_CH2/RTC_GPIO2; no longer U1.GPIO00*/ADC2_CH1/TOUCH1/RTC_GPIO11/CLK_OUT1/EMAC_TX_CLK
- net 3.3V: now also C30.1, D2.A, R10.2, U11.REGIN, U11.VDD, U11.VIO
- net CAN1H: now also JUMPER1.P$1
- net CAN1L: now also R14.2
- net CAN2H: now also JUMPER2.P$1
- net CAN2L: now also R15.2
- net CAN3H: now also JUMPER3.P$1
- net CAN3L: now also R16.2
- net GND: now also C30.2, C31.2, R12.1, R13.1, S1.1, U11.GND
- net N$23: now also R11.1, R12.2, U11.VBUS; no longer F2.1, J2.VBUS
- net RX: now also U11.TXD
- net TX: now also U11.RXD
Other:
- moved on the sheet: A1, C12, C13, J1, J2, L1
